File: Projecte_MiSE/Projecte_MiSE.kicad_sch (KiCad schematic)
At the start: 45 parts, among them IC1 MSP430FR2355TPT, J1 C_DFrobot, J10 Conn_GND_TP, J11 Conn_TXD_TP, J12 Conn_RXD_TP, J2 Conn_SWB, J3 ESP01_WIFI, J4 URM10, J5 Conn_GND_TP, J6 Conn_ACLK_TP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

Commit message: layout and schem pins
Connections:
- net P0: now also IC1.18 (P6.4/TB3.5); no longer IC1.22 (P6.0/TB3.1)
- net P1: now also IC1.19 (P6.3/TB3.4); no longer IC1.21 (P6.1/TB3.2)
- net P12: now also IC1.22 (P6.0/TB3.1); no longer IC1.18 (P6.4/TB3.5)
- net P8: now also IC1.21 (P6.1/TB3.2); no longer IC1.19 (P6.3/TB3.4)
Changed lines of the file:
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@@
+		)
+	)
+	(label "P12"
+		(at 172.72 212.09 270)
+		(effects
+			(font
+				(size 1.27 1.27)
+			)
+			(justify right bottom)
 		)
 	)
@@
 		)
 	)
+	(label "P1"
+		(at 165.1 212.09 270)
+		(effects
+			(font
+				(size 1.27 1.27)
+			)
+			(justify right bottom)
+		)
+	)
 	(label "M_L"
 		(at 228.6 130.81 180)
@@
 		)
 	)
-	(label "P12"
-		(at 162.56 210.82 270)
-		(effects
-			(font
-				(size 1.27 1.27)
-			)
-			(justify right bottom)
-		)
-	)
 	(label "GPIOL"
 		(at 339.09 88.9 0)
@@
 		)
 	)
-	(label "P1"
-		(at 170.18 212.09 270)
-		(effects
-			(font
-				(size 1.27 1.27)
-			)
-			(justify right bottom)
-		)
-	)
 	(label "trg"
 		(at 236.22 171.45 0)
@@
 		)
 	)
+	(label "crystall-"
+		(at 106.68 166.37 180)
+		(effects
+			(font
+				(size 1.27 1.27)
+			)
+			(justify right bottom)
+		)
+	)
+	(label "P1"
+		(at 82.55 260.35 270)
+		(effects
+			(font
+				(size 1.27 1.27)
+			)
+			(justify right bottom)
+		)
+	)
+	(label "L_R"
+		(at 247.65 128.27 270)
+		(effects
+			(font
+				(size 1.27 1.27)
+			)
+			(justify right bottom)
+		)
+	)
+	(label "P8"
+		(at 170.18 212.09 270)
+		(effects
+			(font
+				(size 1.27 1.27)
+			)
+			(justify right bottom)
+		)
+	)
+	(label "SBWTDIO"
+		(at 83.82 151.13 0)
+		(effects
+			(font
+				(size 1.27 1.27)
+				(thickness 0.1588)
+			)
+			(justify left bottom)
+		)
+	)
+	(label "THL"
+		(at 317.5 90.17 180)
+		(effects
+			(font
+				(size 1.27 1.27)
+			)
+			(justify right bottom)
+		)
+	)
+	(label "TXD"
+		(at 210.82 257.81 0)
+		(effects
+			(font
+				(size 1.27 1.27)
+			)
+			(justify left bottom)
+		)
+	)
+	(label "GPIOL"
+		(at 160.02 101.6 90)
+		(effects
+			(font
+				(size 1.27 1.27)
+			)
+			(justify left bottom)
+		)
+	)
+	(label "JSEL"
+		(at 261.62 86.36 180)
+		(effects
+			(font
+				(size 1.27 1.27)
+			)
+			(justify right bottom)
+		)
+	)
 	(label "P2"
 		(at 167.64 212.09 270)
@@
 	)
 	(label "crystall-"
-		(at 106.68 166.37 180)
-		(effects
-			(font
-				(size 1.27 1.27)
-			)
-			(justify right bottom)
-		)
-	)
-	(label "P1"
-		(at 82.55 260.35 270)
-		(effects
-			(font
-				(size 1.27 1.27)
-			)
-			(justify right bottom)
-		)
-	)
-	(label "L_R"
-		(at 247.65 128.27 270)
-		(effects
-			(font
-				(size 1.27 1.27)
-			)
-			(justify right bottom)
-		)
-	)
-	(label "P0"
-		(at 172.72 212.09 270)
-		(effects
-			(font
-				(size 1.27 1.27)
-			)
-			(justify right bottom)
-		)
-	)
-	(label "SBWTDIO"
-		(at 83.82 151.13 0)
-		(effects
-			(font
-				(size 1.27 1.27)
-				(thickness 0.1588)
-			)
-			(justify left bottom)
-		)
-	)
-	(label "THL"
-		(at 317.5 90.17 180)
-		(effects
-			(font
-				(size 1.27 1.27)
-			)
-			(justify right bottom)
-		)
-	)
-	(label "TXD"
-		(at 210.82 257.81 0)
-		(effects
-			(font
-				(size 1.27 1.27)
-			)
-			(justify left bottom)
-		)
-	)
-	(label "GPIOL"
-		(at 160.02 101.6 90)
-		(effects
-			(font
-				(size 1.27 1.27)
-			)
-			(justify left bottom)
-		)
-	)
-	(label "JSEL"
-		(at 261.62 86.36 180)
-		(effects
-			(font
-				(size 1.27 1.27)
-			)
-			(justify right bottom)
-		)
-	)
-	(label "crystall-"
 		(at 38.1 190.5 180)
 		(effects
@@
 		)
 	)
-	(label "P8"
-		(at 165.1 212.09 270)
-		(effects
-			(font
-				(size 1.27 1.27)
-			)
-			(justify right bottom)
-		)
-	)
 	(label "MISO"
 		(at 218.44 158.75 0)
@@
 		)
 	)
+	(label "P0"
+		(at 162.56 210.82 270)
+		(effects
+			(font
+				(size 1.27 1.27)
+			)
+			(justify right bottom)
+		)
+	)

Commit message: relocated pins and added power flags
ERC check
Connections:
- net GPIOD: now also IC1.35 (P3.7/OA3+); no longer IC1.36 (P3.6/OA3-)
- net GPIOL: now also IC1.45 (P3.2/OA2-); no longer IC1.44 (P3.3/OA2+)
- net GPIOR: now also IC1.44 (P3.3/OA2+); no longer IC1.45 (P3.2/OA2-)
- net GPIOU: now also IC1.36 (P3.6/OA3-); no longer IC1.35 (P3.7/OA3+)

Commit message: netclasses
Parts:
- C1, C2: value 15p -> 12p
- R1, R10, R11, R12, R8, R9: value R -> 10k
- R13: value R -> 120
Other:
- moved on the sheet: R7
Changed lines of the file:
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@@
 	(wire
 		(pts
+			(xy 218.44 241.3) (xy 218.44 238.76)
+		)
+		(stroke
+			(width 0)
+			(type default)
+		)
+	)
+	(wire
+		(pts
 			(xy 124.46 241.3) (xy 124.46 242.57)
 		)
@@
 	(wire
 		(pts
-			(xy 218.44 236.22) (xy 218.44 237.49)
+			(xy 218.44 234.95) (xy 218.44 237.49)
 		)
 		(stroke
@@
 	(wire
 		(pts
-			(xy 218.44 255.27) (xy 218.44 246.38)
+			(xy 218.44 255.27) (xy 218.44 248.92)
 		)
 		(stroke
@@
 		(lib_id "Device:R")
 		(at 317.5 78.74 0)
+		(mirror y)
 		(unit 1)
 		(exclude_from_sim no)
@@
 		(dnp no)
 		(property "Reference" "R1"
-			(at 320.04 77.4699 0)
+			(at 314.96 77.4699 0)
 			(effects
 				(font
@@
 			)
 		)
-		(property "Value" "R"
-			(at 320.04 80.0099 0)
+		(property "Value" "10k"
+			(at 314.96 80.0099 0)
 			(effects
 				(font
@@
 		)
 		(property "Footprint" "Resistor_SMD:R_0805_2012Metric"
-			(at 315.722 78.74 90)
+			(at 319.278 78.74 90)
 			(effects
 				(font
@@
 			)
 		)
-		(property "Value" "15p"
+		(property "Value" "12p"
 			(at 57.15 195.5799 0)
 			(effects
@@
 	(symbol
 		(lib_id "power:+3.3V")
-		(at 218.44 236.22 0)
+		(at 218.44 234.95 0)
 		(unit 1)
 		(exclude_from_sim no)
@@
 		(on_board yes)
 		(dnp no)
-		(fields_autoplaced yes)
 		(property "Reference" "#PWR017"
-			(at 218.44 240.03 0)
+			(at 218.44 238.76 0)
 			(effects
 				(font
@@
 		)
 		(property "Value" "+3.3V"
-			(at 218.44 231.14 0)
+			(at 216.154 231.394 0)
 			(effects
 				(font
@@
 		)
 		(property "Footprint" ""
-			(at 218.44 236.22 0)
+			(at 218.44 234.95 0)
 			(effects
 				(font
@@
 		)
 		(property "Datasheet" ""
-			(at 218.44 236.22 0)
+			(at 218.44 234.95 0)
 			(effects
 				(font
@@
 		)
 		(property "Description" "Power symbol creates a global label with name \"+3.3V\""
-			(at 218.44 236.22 0)
+			(at 218.44 234.95 0)
 			(effects
 				(font
@@
 			)
 		)
-		(property "Value" "R"
+		(property "Value" "10k"
 			(at 363.22 80.0099 0)
 			(effects
@@
 			)
 		)
-		(property "Value" "R"
+		(property "Value" "120"
 			(at 251.714 130.556 90)
 			(effects
@@
 			)
 		)
-		(property "Value" "15p"
+		(property "Value" "12p"
 			(at 34.29 195.5799 0)
 			(effects
@@
 		(lib_id "Device:R")
 		(at 317.5 62.23 0)
+		(mirror y)
 		(unit 1)
 		(exclude_from_sim no)
@@
 		(dnp no)
 		(property "Reference" "R8"
-			(at 320.04 60.9599 0)
+			(at 314.96 60.9599 0)
 			(effects
 				(font
@@
 			)
 		)
-		(property "Value" "R"
-			(at 320.04 63.4999 0)
+		(property "Value" "10k"
+			(at 314.96 63.4999 0)
 			(effects
 				(font
@@
 		)
 		(property "Footprint" "Resistor_SMD:R_0805_2012Metric"
-			(at 315.722 62.23 90)
+			(at 319.278 62.23 90)
 			(effects
 				(font
@@
 	(symbol
 		(lib_id "Device:R")
-		(at 218.44 242.57 0)
+		(at 218.44 245.11 0)
 		(unit 1)
 		(exclude_from_sim no)
@@
 		(fields_autoplaced yes)
 		(property "Reference" "R7"
-			(at 220.98 241.2999 0)
+			(at 220.98 243.8399 0)
 			(effects
 				(font
@@
 		)
 		(property "Value" "10k"
-			(at 220.98 243.8399 0)
+			(at 220.98 246.3799 0)
 			(effects
 				(font
@@
 		)
 		(property "Footprint" "Resistor_SMD:R_0805_2012Metric"
-			(at 216.662 242.57 90)
+			(at 216.662 245.11 90)
 			(effects
 				(font
@@
 		)
 		(property "Datasheet" "~"
-			(at 218.44 242.57 0)
+			(at 218.44 245.11 0)
 			(effects
 				(font
@@
 		)
 		(property "Description" "Resistor"
-			(at 218.44 242.57 0)
+			(at 218.44 245.11 0)
 			(effects
 				(font
@@
 		(lib_id "Device:R")
 		(at 365.76 62.23 0)
+		(mirror y)
 		(unit 1)
 		(exclude_from_sim no)
@@
 		(dnp no)
 		(property "Reference" "R10"
-			(at 368.3 60.9599 0)
+			(at 363.22 60.9599 0)
 			(effects
 				(font
@@
 			)
 		)
-		(property "Value" "R"
-			(at 368.3 63.4999 0)
+		(property "Value" "10k"
+			(at 363.22 63.4999 0)
 			(effects
 				(font
@@
 		)
 		(property "Footprint" "Resistor_SMD:R_0805_2012Metric"
-			(at 363.982 62.23 90)
+			(at 367.538 62.23 90)
 			(effects
 				(font
@@
 		(lib_id "Device:R")
 		(at 317.5 102.87 0)
+		(mirror y)
 		(unit 1)
 		(exclude_from_sim no)
@@
 		(dnp no)
 		(property "Reference" "R9"
-			(at 320.04 101.5999 0)
+			(at 314.96 101.5999 0)
 			(effects
 				(font
@@
 			)
 		)
-		(property "Value" "R"
-			(at 320.04 104.1399 0)
+		(property "Value" "10k"
+			(at 314.96 104.1399 0)
 			(effects
 				(font
@@
 		)
 		(property "Footprint" "Resistor_SMD:R_0805_2012Metric"
-			(at 315.722 102.87 90)
+			(at 319.278 102.87 90)
 			(effects
 				(font
@@
 		(lib_id "Device:R")
 		(at 365.76 97.79 0)
+		(mirror y)
 		(unit 1)
 		(exclude_from_sim no)
@@
 		(dnp no)
 		(property "Reference" "R12"
-			(at 368.3 96.5199 0)
+			(at 363.22 96.5199 0)
 			(effects
 				(font
@@
 			)
 		)
-		(property "Value" "R"
-			(at 368.3 99.0599 0)
+		(property "Value" "10k"
+			(at 363.22 99.0599 0)
 			(effects
 				(font
@@
 		)
 		(property "Footprint" "Resistor_SMD:R_0805_2012Metric"
-			(at 363.982 97.79 90)
+			(at 367.538 97.79 90)
 			(effects
 				(font
