File: Projecte_MiSE/Projecte_MiSE.kicad_sch (KiCad schematic)
At the start: 45 parts, among them IC1 MSP430FR2355TPT, J1 C_DFrobot, J10 Conn_GND_TP, J11 Conn_TXD_TP, J12 Conn_RXD_TP, J2 Conn_SWB, J3 ESP01_WIFI, J4 URM10, J5 Conn_GND_TP, J6 Conn_ACLK_TP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

Commit message: Routing correction
Other:
- title: Placa projecte MiSE -> PCB projecte MiSE
Changed lines of the file:
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@@
 	(paper "A3")
 	(title_block
-		(title "Placa projecte MiSE")
-		(date "2026-03-10")
-		(rev "4/4")
+		(title "PCB projecte MiSE")
+		(date "2026-03-15")
+		(rev "5/5")
+		(comment 1 "K. Brandon Ventura L.")
+		(comment 2 "Raúl Casado Luque")
 	)
 	(rectangle
